File: EDA files/EEZ DIB MUX14D r1B2.sch (EAGLE design)
At the start: 55 parts, among them IC1 M24C32-WMN6P, IC2 74HC1G126GW,125, IC3 LP2985-33DBVR, IC4 STM32F030C6T6, IC5 ULN2803ADWR, IC6 ULN2803ADWR, K1 3572.1220.051, K10 3572.1220.051, K11 3572.1220.051, K12 3572.1220.051, K13 3572.1220.051, K14 3572.1220.051, K15 3572.1220.051, K16 3572.1220.051, K17 3572.1220.051, K2 3572.1220.051, K3 3572.1220.051, K4 3572.1220.051, K5 3572.1220.051, K6 3572.1220.051, K7 3572.1220.051, K8 3572.1220.051, K9 3572.1220.051, Q1 2N7002, X1 DS1014-10RF1B, X2 77317-104-28LF, X3 DS1014-10RF1B, X4 N.C., X5 691327310016, X6 691327310016

Commit message: ADIB ID=002
Connections:
- new net N$1: X1-10.1, X1-9.1
- new net N$2: X3-10.1, X3-9.1
Other:
- note added: "ADIB1_ID=002"
- note added: "ADIB2_ID=002"
Changed lines of the file:
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@@
 <setting verticaltext="up"/>
 </settings>
-<grid distance="0.1" unitdist="inch" unit="inch" style="lines" multiple="1" display="no" altdistance="0.01" altunitdist="inch" altunit="inch"/>
+<grid distance="0.025" unitdist="inch" unit="inch" style="lines" multiple="4" display="no" altdistance="0.01" altunitdist="inch" altunit="inch"/>
 <layers>
 <layer number="1" name="Top" color="4" fill="1" visible="no" active="no"/>
@@
 <text x="7.62" y="88.9" size="1.778" layer="97" rot="MR180">ADIB connectors</text>
 <wire x1="142.24" y1="91.44" x2="5.08" y2="91.44" width="0.1524" layer="97" style="shortdash"/>
+<text x="27.94" y="66.675" size="1.4224" layer="103">ADIB1_ID=002</text>
+<text x="81.28" y="66.675" size="1.4224" layer="103">ADIB2_ID=002</text>
 </plain>
 <instances>
@@
 </segment>
 </net>
+<net name="N$1" class="0">
+<segment>
+<pinref part="X1" gate="-9" pin="1"/>
+<wire x1="30.48" y1="71.12" x2="27.94" y2="71.12" width="0.1524" layer="91"/>
+<wire x1="27.94" y1="71.12" x2="27.94" y2="68.58" width="0.1524" layer="91"/>
+<wire x1="27.94" y1="68.58" x2="58.42" y2="68.58" width="0.1524" layer="91"/>
+<wire x1="58.42" y1="68.58" x2="58.42" y2="71.12" width="0.1524" layer="91"/>
+<pinref part="X1" gate="-10" pin="1"/>
+<wire x1="58.42" y1="71.12" x2="55.88" y2="71.12" width="0.1524" layer="91"/>
+</segment>
+</net>
+<net name="N$2" class="0">
+<segment>
+<pinref part="X3" gate="-9" pin="1"/>
+<wire x1="83.82" y1="71.12" x2="81.28" y2="71.12" width="0.1524" layer="91"/>
+<wire x1="81.28" y1="71.12" x2="81.28" y2="68.58" width="0.1524" layer="91"/>
+<wire x1="81.28" y1="68.58" x2="111.76" y2="68.58" width="0.1524" layer="91"/>
+<wire x1="111.76" y1="68.58" x2="111.76" y2="71.12" width="0.1524" layer="91"/>
+<pinref part="X3" gate="-10" pin="1"/>
+<wire x1="111.76" y1="71.12" x2="109.22" y2="71.12" width="0.1524" layer="91"/>
+</segment>
+</net>

Commit message: small PCB layout corrections
Parts:
- added C11: 10n, rcl:C-EUC0805
- added C12, C13: 100n, rcl:C-EUC0603
- added C14: 100p, rcl:C-EUC0805
- added IC7, IC8: ULN2803ADWR, EEZ_TI:ULN2803ADWR
- added R3: 1K5, rcl:R-EU_R0805
- added R4, R5: 30K, rcl:R-EU_R0805
- added R6: 120K, rcl:R-EU_R0805
- added R7: 100K, rcl:R-EU_R0805
- C1: value EEEFK1V470P -> 100n; device EEZ_Lib1:ECAPPANASONIC_H -> rcl:C-EUC0603
- C10, C2: value 100n -> 2u2; device rcl:C-EUC0603 -> rcl:C-EUC0805
- C3: value 2u2 -> EEEFK1V470P; device rcl:C-EUC0805 -> EEZ_Lib1:ECAPPANASONIC_H
- C4: value 10n -> 100n; device rcl:C-EUC0805 -> rcl:C-EUC0603
- C8: value 2u2 -> ???
- IC1: value M24C32-WMN6P -> STM32F030C6T6; device EEZ_Lib1:AT24CXXSOIC8 -> EEZ_DIB:STM32F030C6T6
- IC3: value LP2985-33DBVR -> M24C32-WMN6P; device EEZ_DIB:LP2985 -> EEZ_Lib1:AT24CXXSOIC8
- IC4: value STM32F030C6T6 -> LP2985-33DBVR; device EEZ_DIB:STM32F030C6T6 -> EEZ_DIB:LP2985
- IC5: value ULN2803ADWR -> TLV9001IDBVR; device EEZ_TI:ULN2803ADWR -> EEZ_TI:OPA376AIDBVR
- IC6: value ULN2803ADWR -> LM335; device EEZ_TI:ULN2803ADWR -> EEZ_TI:LM335-TO92
- R2: value 100K -> ???
- X1: value DS1014-10RF1B -> N.C.; device EEZ_connectors:DS1014-10RF1B -> con-samtec:SSW-106-02-S-S
- X4: value N.C. -> DS1014-10RF1B; device con-samtec:SSW-106-02-S-S -> EEZ_connectors:DS1014-10RF1B
Connections:
- removed net N$1 (its old number): X1-10.1, X1-9.1
- new net CJ_AIN: C14.2, C8.2, IC5A.OUT, R2.2, R6.1
- new net N$183: C14.1, IC5A.-IN, R5.1, R6.2
- new net N$184: IC5A.+IN, R4.1
- new net N$2: X4-10.1, X4-9.1
- new net N$3: IC6.C, R3.2, R4.2
- new net N$6: IC1.PA7, R2.1
- net +3V3: now also C1.2, C2.1, C4.1, C5.2, C7.2, IC1.VDDA, IC1.VDD_1, IC1.VDD_2, IC1.VDD_3, IC3.VCC, IC4.OUT, R5.2; no longer C10.2, C2.2, C5.1, C7.1, C8.2, IC1.VCC, IC3.OUT, IC4.VDDA, IC4.VDD_1, IC4.VDD_2, IC4.VDD_3
- net +5V: now also C10.2, C12.1, C13.1, C3.+, IC4.IN, IC4.ON/!OFF, IC5P.V+, R3.1; no longer C1.+, C3.2, IC3.IN, IC3.ON/!OFF
- net BOOT0: now also IC1.BOOT0; no longer IC4.BOOT0
- net DIB_A0: now also IC3.A0; no longer IC1.A0
- net DIB_A1: now also IC3.A1; no longer IC1.A1
- net DIB_A2: now also IC3.A2; no longer IC1.A2
- net DIB_CSA: now also IC1.PB12; no longer IC4.PB12
- net DIB_MISO: now also IC1.PB14; no longer IC4.PB14
- net DIB_MOSI: now also IC1.PB15; no longer IC4.PB15
- net DIB_NRESET: now also IC1.NRST; no longer IC4.NRST
- net DIB_SCL: now also IC3.SCL; no longer IC1.SCL
- net DIB_SCLK: now also IC1.PB13; no longer IC4.PB13
- net DIB_SDA: now also IC3.SDA; no longer IC1.SDA
- net DIB_SYNC: now also IC1.PC15-OSC32_OUT; no longer IC4.PC15-OSC32_OUT
- net GND: now also C1.1, C11.1, C12.2, C13.2, C2.2, C3.-, C4.2, C5.1, C7.1, IC1.VSSA, IC1.VSS_1, IC1.VSS_3, IC3.WP, IC4.GND, IC5P.V-, IC6.A, IC7.GND, IC8.GND, R7.2, X1-3.1; no longer C1.-, C2.1, C3.1, C4.1, C5.2, C7.2, IC1.GND, IC1.WP, IC4.VSSA, IC4.VSS_1, IC4.VSS_3, IC5.GND, IC6.GND, R2.2, X4-3.1
- net N$28: now also IC7.COM; no longer IC5.COM
- net N$30: now also IC7.1C; no longer IC5.1C
- net N$32: now also IC7.2C, K31.2; no longer IC5.2C, K21.2
- net N$34: now also IC7.3C, K61.2; no longer IC5.3C, K31.2
- net N$35: now also IC7.4C, K81.2; no longer IC5.4C, K41.2
- net N$36: now also IC7.5C, K121.2; no longer IC5.5C, K51.2
- net N$38: now also IC7.6C, K141.2; no longer IC5.6C, K61.2
- net N$40: now also IC7.7C, K161.2; no longer IC5.7C, K71.2
- net N$42: now also IC7.8C; no longer IC5.8C
- net N$43: now also K51.2; no longer K81.2
- net N$44: now also IC8.COM; no longer IC6.COM
- net N$46: now also IC8.1C, K21.2; no longer IC6.1C, K101.2
- net N$48: now also IC8.2C, K41.2; no longer IC6.2C, K111.2
- net N$50: now also IC8.3C, K71.2; no longer IC6.3C, K121.2
- net N$52: now also IC8.4C, K101.2; no longer IC6.4C, K131.2
- net N$54: now also IC8.5C, K131.2; no longer IC6.5C, K141.2
- net N$56: now also IC8.6C; no longer IC6.6C
- net N$58: now also IC8.7C, K171.2; no longer IC6.7C, K161.2
- net N$60: now also IC8.8C, K111.2; no longer IC6.8C, K171.2
- net N$70: now also C11.2, IC4.BYPASS; no longer C4.2, IC3.BYPASS
- net N$75: now also IC1.PA12; no longer IC4.PA12
- net P1: now also IC1.PB10, IC7.8B; no longer IC4.PA7, IC5.8B
- net P1H: now also K122.S, K142.S, K162.S; no longer K22.S, K42.S, K72.S
- net P1H.2: now also K32.P; no longer K22.P
- net P1H.3: now also K62.P; no longer K32.P
- net P1H.4: now also K82.P; no longer K42.P
- net P1H.5: now also K122.P; no longer K52.P
- net P1H.6: now also K142.P; no longer K62.P
- net P1H.7: now also K162.P; no longer K72.P
- net P1H_OUT: now also X3-4.1; no longer X1-4.1
- net P1L: now also K123.S, K143.S, K163.S; no longer K23.S, K43.S, K73.S
- net P1L.2: now also K33.P; no longer K23.P
- net P1L.3: now also K63.P; no longer K33.P
- net P1L.4: now also K83.P; no longer K43.P
- net P1L.5: now also K123.P; no longer K53.P
- net P1L.6: now also K143.P; no longer K63.P
- net P1L.7: now also K163.P; no longer K73.P
- net P1L_OUT: now also X3-3.1; no longer X1-3.1
- net P2: now also IC1.PB7, IC8.8B; no longer IC4.PB7, IC6.8B
- net P2H: now also K22.S, K42.S, K52.P, K72.S; no longer K122.S, K142.S, K162.S, K82.P
- net P2H.1: now also K22.P; no longer K102.P
- net P2H.2: now also K42.P; no longer K112.P
- net P2H.3: now also K72.P; no longer K122.P
- net P2H.4: now also K102.P; no longer K132.P
- net P2H.5: now also K132.P; no longer K142.P
- net P2H.7: now also K172.P; no longer K162.P
- net P2H_OUT: now also K112.P, X4-4.1; no longer K172.P, X3-4.1
- net P2L: now also K23.S, K43.S, K53.P, K73.S; no longer K123.S, K143.S, K163.S, K83.P
- net P2L.1: now also K23.P; no longer K103.P
- net P2L.2: now also K43.P; no longer K113.P
- net P2L.3: now also K73.P; no longer K123.P
- net P2L.4: now also K103.P; no longer K133.P
- net P2L.5: now also K133.P; no longer K143.P
- net P2L.6: now also K173.P; no longer K163.P
- net P2L_OUT: now also K113.P, X4-3.1; no longer K173.P, X3-3.1
- net P2_EXT: now also IC1.PA15, R7.1; no longer IC4.PA15, R2.1
- net PORT_A0: now also IC1.PA0, IC7.1B; no longer IC4.PA0, IC5.1B
- net PORT_A1: now also IC1.PA1, IC7.2B; no longer IC4.PA1, IC5.2B
- net PORT_A2: now also IC1.PA2, IC7.3B; no longer IC4.PA2, IC5.3B
- net PORT_A3: now also IC1.PA3, IC7.4B; no longer IC4.PA3, IC5.4B
- net PORT_A4: now also IC1.PA4, IC7.5B; no longer IC4.PA4, IC5.5B
- net PORT_A5: now also IC1.PA5, IC7.6B; no longer IC4.PA5, IC5.6B
- net PORT_A6: now also IC1.PA6, IC7.7B; no longer IC4.PA6, IC5.7B
- net PORT_B0: now also IC1.PB0, IC8.1B; no longer IC4.PB0, IC6.1B
- net PORT_B1: now also IC1.PB1, IC8.2B; no longer IC4.PB1, IC6.2B
- net PORT_B2: now also IC1.PB2, IC8.3B; no longer IC4.PB2, IC6.3B
- net PORT_B3: now also IC1.PB3, IC8.4B; no longer IC4.PB3, IC6.4B
- net PORT_B4: now also IC1.PB4, IC8.5B; no longer IC4.PB4, IC6.5B
- net PORT_B5: now also IC1.PB5, IC8.6B; no longer IC4.PB5, IC6.6B
- net PORT_B6: now also IC1.PB6, IC8.7B; no longer IC4.PB6, IC6.7B
- net SWCLK: now also IC1.PA14, X1-2.1; no longer IC4.PA14, X4-2.1
- net SWDIO: now also IC1.PA13, X1-4.1; no longer IC4.PA13, X4-4.1
- net UART_RX: now also IC1.PA10; no longer IC4.PA10
- net UART_TX: now also IC1.PA9; no longer IC4.PA9
Other:
- moved on the sheet: C10, C2, C4, C5, C6, C7, C8, C9, K1, K10, K11, K12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

Commit message: PCB ID added
Connections:
- new net N$7: IC1.PF0-OSC_IN
- net GND: now also IC1.PF1-OSC_OUT
Other:
- note added: "ADIB1_ID=2"
- note added: "ADIB2_ID=2"
- note added: "PCB_ID0"
- note added: "PCB_ID1"
- note added: "PCB_ID=2"
- note added: "Power consumption per relay: 35 mA / 175 mW Max. consumption: 2.8 W"
- note removed: "ADIB1_ID=002"
- note removed: "ADIB2_ID=002"
Changed lines of the file:
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@@
 <text x="7.62" y="88.9" size="1.778" layer="97" rot="MR180">ADIB connectors</text>
 <wire x1="142.24" y1="91.44" x2="5.08" y2="91.44" width="0.1524" layer="97" style="shortdash"/>
-<text x="27.94" y="66.675" size="1.4224" layer="103">ADIB1_ID=002</text>
-<text x="81.28" y="66.675" size="1.4224" layer="103">ADIB2_ID=002</text>
+<text x="27.94" y="66.675" size="1.4224" layer="103">ADIB1_ID=2</text>
+<text x="81.28" y="66.675" size="1.4224" layer="103">ADIB2_ID=2</text>
+<text x="162.56" y="109.855" size="1.27" layer="103">PCB_ID0</text>
+<text x="162.56" y="107.315" size="1.27" layer="103">PCB_ID1</text>
+<text x="144.78" y="109.855" size="1.27" layer="103">PCB_ID=2</text>
 </plain>
 <instances>
@@
 <wire x1="162.56" y1="101.6" x2="162.56" y2="99.06" width="0.1524" layer="91"/>
 <pinref part="C6" gate="G$1" pin="2"/>
-<wire x1="162.56" y1="101.6" x2="157.48" y2="101.6" width="0.1524" layer="91"/>
+<wire x1="162.56" y1="101.6" x2="160.02" y2="101.6" width="0.1524" layer="91"/>
+<wire x1="160.02" y1="101.6" x2="157.48" y2="101.6" width="0.1524" layer="91"/>
 <wire x1="157.48" y1="101.6" x2="157.48" y2="99.06" width="0.1524" layer="91"/>
 <junction x="162.56" y="101.6"/>
@@
 <pinref part="TP1" gate="G$1" pin="P$1"/>
 <wire x1="157.48" y1="104.14" x2="157.48" y2="101.6" width="0.1524" layer="91"/>
+<pinref part="IC1" gate="G$1" pin="PF1-OSC_OUT"/>
+<wire x1="175.26" y1="106.68" x2="160.02" y2="106.68" width="0.1524" layer="91"/>
+<wire x1="160.02" y1="106.68" x2="160.02" y2="101.6" width="0.1524" layer="91"/>
+<junction x="160.02" y="101.6"/>
 </segment>
 <segment>
@@
 <wire x1="210.82" y1="78.74" x2="210.82" y2="66.04" width="0.1524" layer="91"/>
 <label x="210.185" y="66.675" size="1.27" layer="102" rot="R90"/>
+</segment>
+</net>
+<net name="N$7" class="0">
+<segment>
+<pinref part="IC1" gate="G$1" pin="PF0-OSC_IN"/>
+<wire x1="175.26" y1="109.22" x2="162.56" y2="109.22" width="0.1524" layer="91"/>
 </segment>
 </net>
@@
 <text x="2.54" y="4.445" size="1.27" layer="94">More info at http://www.envox.hr/eez</text>
 <text x="164.465" y="26.67" size="2.54" layer="94" font="vector">Switch matrix relays control</text>
+<text x="83.185" y="161.29" size="1.27" layer="103">Power consumption per relay: 35 mA / 175 mW
+Max. consumption: 2.8 W</text>
 </plain>
 <instances>
@@
 </schematic>
 </drawing>
+<compatibility>
+<note version="6.3" minversion="6.2.2" severity="warning">
+Since Version 6.2.2 text objects can contain more than one line,
+which will not be processed correctly with this version.
+</note>
+</compatibility>
 </eagle>
