File: EDA files/EEZ DIB MUX14D r1B3.brd (EAGLE design)
At the start: 131 x 95 mm, 67 parts, among them IC1 STM32F030C6T6, IC2 74HC1G126GW,125, IC3 M24C32-WMN6P, IC4 LP2985-33DBVR, IC5 TLV9001IDBVR, IC6 LM335, IC7 ULN2803ADWR, IC8 ULN2803ADWR, K1 3572.1220.051, K10 3572.1220.051, K11 3572.1220.051, K12 3572.1220.051, K13 3572.1220.051, K14 3572.1220.051, K15 3572.1220.051, K16 3572.1220.051, K17 3572.1220.051, K2 3572.1220.051, K3 3572.1220.051, K4 3572.1220.051, K5 3572.1220.051, K6 3572.1220.051, K7 3572.1220.051, K8 3572.1220.051, K9 3572.1220.051, Q1 2N7002, X1 N.C., X2 77317-104-28LF, X3 DS1014-10RF1B, X4 DS1014-10RF1B, X5 691327310016, X6 691327310016

Commit message: Centroid files
Parts:
- removed C8: ???, rcl:C0805
- removed R2: ???, rcl:R0805
- IC5: value TLV9001IDBVR -> MCP6001RT-I/OT
- R4, R5: value 30K -> 10K
- R6: value 120K -> 40K2
- moved C12 3.05 mm to (21.4, 15.3)
- moved IC6 3.05 mm to (12.0, 15.5)
- moved R3 3.05 mm to (17.8, 15.3)
Connections:
- removed net N$6: IC1.17, R2.1
- net CJ_AIN: now also IC1.17; no longer C8.2, R2.2
- net GND: no longer C8.1
Routing:
- net N$6: track 6.45 -> 0.00 mm
- net CJ_AIN: track 83.9 -> 89.9 mm
- net +5V: track 622.3 -> 619.2 mm
- net N$3: track 34.4 -> 31.4 mm
- net GND: track 35.7 -> 34.7 mm, vias 30 -> 29
Other:
- board text added: "EEZ DIB MUX14D (04/2021 r1B3)"
- board text added: "EEZ DIB MUX14D (04/2021 r1B3) Project source code: github.com/eez-open"
- board text removed: "EEZ DIB MUX14D (01/2021 r1B2)"
- board text removed: "EEZ DIB MUX14D (01/2021 r1B2) Project source code: github.com/eez-open"

Commit message: BOM update
Parts:
- IC5: value MCP6001RT-I/OT -> MCP6001T-I/OT
- IC6: value LM335 -> LM335AZ
Changed lines of the file:
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@@
 <grid distance="10" unitdist="mil" unit="mil" style="lines" multiple="10" display="no" altdistance="2.5" altunitdist="mil" altunit="mil"/>
 <layers>
-<layer number="1" name="Top" color="3" fill="1" visible="yes" active="yes"/>
+<layer number="1" name="Top" color="3" fill="1" visible="no" active="yes"/>
 <layer number="2" name="Route2" color="1" fill="3" visible="no" active="no"/>
 <layer number="3" name="Route3" color="4" fill="3" visible="no" active="no"/>
@@
 <layer number="14" name="Route14" color="1" fill="6" visible="no" active="no"/>
 <layer number="15" name="Route15" color="4" fill="6" visible="no" active="no"/>
-<layer number="16" name="Bottom" color="1" fill="1" visible="yes" active="yes"/>
-<layer number="17" name="Pads" color="14" fill="1" visible="yes" active="yes"/>
-<layer number="18" name="Vias" color="6" fill="1" visible="yes" active="yes"/>
-<layer number="19" name="Unrouted" color="6" fill="1" visible="yes" active="yes"/>
+<layer number="16" name="Bottom" color="1" fill="1" visible="no" active="yes"/>
+<layer number="17" name="Pads" color="14" fill="1" visible="no" active="yes"/>
+<layer number="18" name="Vias" color="6" fill="1" visible="no" active="yes"/>
+<layer number="19" name="Unrouted" color="6" fill="1" visible="no" active="yes"/>
 <layer number="20" name="Dimension" color="12" fill="1" visible="yes" active="yes"/>
 <layer number="21" name="tPlace" color="7" fill="1" visible="yes" active="yes"/>
 <layer number="22" name="bPlace" color="6" fill="1" visible="no" active="yes"/>
-<layer number="23" name="tOrigins" color="15" fill="1" visible="yes" active="yes"/>
+<layer number="23" name="tOrigins" color="15" fill="1" visible="no" active="yes"/>
 <layer number="24" name="bOrigins" color="15" fill="1" visible="no" active="yes"/>
 <layer number="25" name="tNames" color="7" fill="1" visible="yes" active="yes"/>
 <layer number="26" name="bNames" color="5" fill="1" visible="no" active="yes"/>
-<layer number="27" name="tValues" color="10" fill="1" visible="no" active="yes"/>
+<layer number="27" name="tValues" color="14" fill="1" visible="yes" active="yes"/>
 <layer number="28" name="bValues" color="10" fill="1" visible="no" active="yes"/>
 <layer number="29" name="tStop" color="7" fill="1" visible="yes" active="yes"/>
@@
 <layer number="41" name="tRestrict" color="4" fill="10" visible="no" active="yes"/>
 <layer number="42" name="bRestrict" color="1" fill="10" visible="no" active="yes"/>
-<layer number="43" name="vRestrict" color="2" fill="10" visible="yes" active="yes"/>
+<layer number="43" name="vRestrict" color="2" fill="10" visible="no" active="yes"/>
 <layer number="44" name="Drills" color="7" fill="1" visible="no" active="yes"/>
 <layer number="45" name="Holes" color="7" fill="1" visible="no" active="yes"/>
@@
 <attribute name="VALUE" x="111.3155" y="73.66" size="1.016" layer="27" ratio="10" rot="R90" align="center"/>
 </element>
-<element name="IC6" library="EEZ_TI" package="TO92" value="LM335" x="11.9507" y="15.494" smashed="yes" rot="R180">
+<element name="IC6" library="EEZ_TI" package="TO92" value="LM335AZ" x="11.9507" y="15.494" smashed="yes" rot="R180">
 <attribute name="NAME" x="5.3848" y="14.8209" size="1.27" layer="25" ratio="10"/>
 <attribute name="VALUE" x="9.0932" y="14.8336" size="1.27" layer="27" ratio="10"/>
@@
 <attribute name="VALUE" x="19.7993" y="14.9225" size="1.016" layer="27" ratio="10"/>
 </element>
-<element name="IC5" library="EEZ_TI" package="DBV5" value="MCP6001RT-I/OT" x="46.8376" y="14.2494" smashed="yes">
+<element name="IC5" library="EEZ_TI" package="DBV5" value="MCP6001T-I/OT" x="46.8376" y="14.2494" smashed="yes">
 <attribute name="NAME" x="45.6946" y="11.4046" size="1.016" layer="25" ratio="10"/>
 <attribute name="VALUE" x="44.0436" y="13.7414" size="0.6096" layer="27" ratio="10"/>

Commit message: #1
Connections:
- net P1 renamed P1.C
- net P2 renamed P2.C
- net P2L.6: now also K15.8; no longer K17.8
- net P2L.7: now also K17.8; no longer K15.8
Routing:
- net P2L.6: track 50.5 -> 29.5 mm
- net P2L.7: track 40.2 -> 60.2 mm
- net N$38: track 87.8 -> 88.6 mm
Other:
- board text added: "EEZ DIB MUX14D (05/2021 r1B3)"
- board text added: "EEZ DIB MUX14D (05/2021 r1B3) Project source code: github.com/eez-open"
- board text removed: "EEZ DIB MUX14D (04/2021 r1B3)"
- board text removed: "EEZ DIB MUX14D (04/2021 r1B3) Project source code: github.com/eez-open"
Changed lines of the file:
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@@
 <setting verticaltext="up"/>
 </settings>
-<grid distance="10" unitdist="mil" unit="mil" style="lines" multiple="10" display="no" altdistance="2.5" altunitdist="mil" altunit="mil"/>
+<grid distance="0.5" unitdist="mil" unit="mil" style="lines" multiple="10" display="no" altdistance="2.5" altunitdist="mil" altunit="mil"/>
 <layers>
-<layer number="1" name="Top" color="3" fill="1" visible="no" active="yes"/>
+<layer number="1" name="Top" color="3" fill="1" visible="yes" active="yes"/>
 <layer number="2" name="Route2" color="1" fill="3" visible="no" active="no"/>
 <layer number="3" name="Route3" color="4" fill="3" visible="no" active="no"/>
@@
 <layer number="14" name="Route14" color="1" fill="6" visible="no" active="no"/>
 <layer number="15" name="Route15" color="4" fill="6" visible="no" active="no"/>
-<layer number="16" name="Bottom" color="1" fill="1" visible="no" active="yes"/>
-<layer number="17" name="Pads" color="14" fill="1" visible="no" active="yes"/>
-<layer number="18" name="Vias" color="6" fill="1" visible="no" active="yes"/>
-<layer number="19" name="Unrouted" color="6" fill="1" visible="no" active="yes"/>
+<layer number="16" name="Bottom" color="1" fill="1" visible="yes" active="yes"/>
+<layer number="17" name="Pads" color="14" fill="1" visible="yes" active="yes"/>
+<layer number="18" name="Vias" color="6" fill="1" visible="yes" active="yes"/>
+<layer number="19" name="Unrouted" color="6" fill="1" visible="yes" active="yes"/>
 <layer number="20" name="Dimension" color="12" fill="1" visible="yes" active="yes"/>
 <layer number="21" name="tPlace" color="7" fill="1" visible="yes" active="yes"/>
-<layer number="22" name="bPlace" color="6" fill="1" visible="no" active="yes"/>
-<layer number="23" name="tOrigins" color="15" fill="1" visible="no" active="yes"/>
+<layer number="22" name="bPlace" color="6" fill="1" visible="yes" active="yes"/>
+<layer number="23" name="tOrigins" color="15" fill="1" visible="yes" active="yes"/>
 <layer number="24" name="bOrigins" color="15" fill="1" visible="no" active="yes"/>
 <layer number="25" name="tNames" color="7" fill="1" visible="yes" active="yes"/>
 <layer number="26" name="bNames" color="5" fill="1" visible="no" active="yes"/>
-<layer number="27" name="tValues" color="14" fill="1" visible="yes" active="yes"/>
+<layer number="27" name="tValues" color="14" fill="1" visible="no" active="yes"/>
 <layer number="28" name="bValues" color="10" fill="1" visible="no" active="yes"/>
 <layer number="29" name="tStop" color="7" fill="1" visible="yes" active="yes"/>
@@
 <dimension x1="-10" y1="81" x2="-11" y2="17" x3="-12" y3="49" textsize="2" layer="47" dtype="vertical"/>
 <text x="112.6263" y="82.5206" size="1.27" layer="21" font="vector" ratio="10" rot="SR0">EEZ DIB MUX14D
-(04/2021 r1B3)</text>
-<text x="129.2946" y="90.0898" size="1.27" layer="22" font="vector" ratio="10" rot="SMR0">EEZ DIB MUX14D (04/2021 r1B3)
+(05/2021 r1B3)</text>
+<text x="129.2946" y="90.0898" size="1.27" layer="22" font="vector" ratio="10" rot="SMR0">EEZ DIB MUX14D (05/2021 r1B3)
 Project source code: github.com/eez-open</text>
 <rectangle x1="106.6038" y1="86.9061" x2="128.7018" y2="92.5576" layer="21"/>
@@
 <wire x1="109.5629" y1="60.7695" x2="107.7595" y2="60.7695" width="0.2032" layer="1"/>
 <wire x1="47.244" y1="31.242" x2="49.784" y2="33.782" width="0.2032" layer="1"/>
-<wire x1="49.784" y1="33.782" x2="49.784" y2="37.2999" width="0.2032" layer="1"/>
-<via x="49.784" y="37.2999" extent="1-16" drill="0.4" shape="octagon"/>
-<wire x1="49.784" y1="37.2999" x2="51.181" y2="38.6969" width="0.2032" layer="16"/>
+<via x="49.784" y="38.6969" extent="1-16" drill="0.4" shape="octagon"/>
 <via x="104.7242" y="38.6969" extent="1-16" drill="0.4" shape="octagon"/>
-<wire x1="104.7242" y1="38.6969" x2="51.181" y2="38.6969" width="0.2032" layer="16"/>
+<wire x1="104.7242" y1="38.6969" x2="49.784" y2="38.6969" width="0.2032" layer="16"/>
 <wire x1="105.029" y1="58.039" x2="105.029" y2="39.0017" width="0.2032" layer="1"/>
 <wire x1="105.029" y1="39.0017" x2="104.7242" y2="38.6969" width="0.2032" layer="1"/>
 <wire x1="107.7595" y1="60.7695" x2="105.029" y2="58.039" width="0.2032" layer="1"/>
+<wire x1="49.784" y1="33.782" x2="49.784" y2="38.6969" width="0.2032" layer="1"/>
 </signal>
 <signal name="N$40">
@@
 <contactref element="K10" pad="14"/>
 <contactref element="K4" pad="14"/>
-<contactref element="K17" pad="14"/>
-<contactref element="K15" pad="14"/>
 <contactref element="X6" pad="8"/>
 <contactref element="K11" pad="14"/>
@@
 <wire x1="43.2435" y1="59.3725" x2="40.4495" y2="59.3725" width="0.4064" layer="16"/>
 <wire x1="40.4495" y1="59.3725" x2="38.862" y2="60.96" width="0.4064" layer="16"/>
-<wire x1="59.944" y1="34.4805" x2="42.291" y2="34.4805" width="0.4064" layer="16"/>
-<wire x1="59.944" y1="36.068" x2="59.944" y2="34.4805" width="0.4064" layer="16"/>
-<wire x1="59.944" y1="34.4805" x2="79.4385" y2="34.4805" width="0.4064" layer="16"/>
-<wire x1="79.4385" y1="34.4805" x2="81.026" y2="36.068" width="0.4064" layer="16"/>
+<wire x1="42.291" y1="34.4805" x2="59.9567" y2="34.4805" width="0.4064" layer="16"/>
 <via x="42.291" y="34.4805" extent="1-16" drill="0.4" shape="octagon"/>
+<wire x1="59.9567" y1="34.4805" x2="79.4385" y2="34.4805" width="0.4064" layer="16"/>
 <wire x1="42.291" y1="34.4805" x2="42.291" y2="24.765" width="0.4064" layer="1"/>
 <wire x1="42.291" y1="34.4805" x2="40.4495" y2="34.4805" width="0.4064" layer="16"/>
 <wire x1="40.4495" y1="34.4805" x2="38.862" y2="36.068" width="0.4064" layer="16"/>
-<wire x1="61.468" y1="37.592" x2="59.944" y2="36.068" width="0.4064" layer="1"/>
 <wire x1="18.35" y1="19.665" x2="37.191" y2="19.665" width="0.4064" layer="1"/>
 <wire x1="37.191" y1="19.665" x2="42.291" y2="24.765" width="0.4064" layer="1"/>
@@
 <wire x1="82.4865" y1="71.9455" x2="82.4865" y2="62.4205" width="0.4064" layer="1"/>
 <wire x1="81.026" y1="60.96" x2="82.4865" y2="62.4205" width="0.4064" layer="1"/>
+<contactref element="K15" pad="14"/>
+<contactref element="K17" pad="14"/>
+<wire x1="79.4385" y1="34.4805" x2="81.026" y2="36.068" width="0.4064" layer="16"/>
+<wire x1="59.944" y1="36.068" x2="59.944" y2="34.4932" width="0.4064" layer="16"/>
+<wire x1="59.944" y1="34.4932" x2="59.9567" y2="34.4805" width="0.4064" layer="16"/>
+<wire x1="61.468" y1="37.592" x2="59.944" y2="36.068" width="0.4064" layer="1"/>
 </signal>
 <signal name="P2L.1">
@@
 <signal name="P2L.6">
 <contactref element="X6" pad="4"/>
-<contactref element="K17" pad="8"/>
 <wire x1="18.35" y1="34.905" x2="18.9142" y2="34.3408" width="0.4064" layer="16"/>
-<via x="65.786" y="33.528" extent="1-16" drill="0.4" shape="octagon"/>
-<wire x1="18.9142" y1="34.3408" x2="29.8958" y2="34.3408" width="0.4064" layer="16"/>
-<wire x1="29.8958" y1="34.3408" x2="31.1912" y2="34.3408" width="0.4064" layer="16"/>
-<wire x1="65.786" y1="36.068" x2="65.786" y2="33.528" width="0.4064" layer="1"/>
-<wire x1="65.786" y1="33.528" x2="33.7693" y2="33.528" width="0.4064" layer="16"/>
+<via x="44.704" y="33.528" extent="1-16" drill="0.4" shape="octagon"/>
+<wire x1="18.9142" y1="34.3408" x2="32.9565" y2="34.3408" width="0.4064" layer="16"/>
 <wire x1="33.7693" y1="33.528" x2="32.9565" y2="34.3408" width="0.4064" layer="16"/>
-<wire x1="32.9565" y1="34.3408" x2="31.1912" y2="34.3408" width="0.4064" layer="16"/>
+<contactref element="K15" pad="8"/>
+<wire x1="33.7693" y1="33.528" x2="44.704" y2="33.528" width="0.4064" layer="16"/>
+<wire x1="44.704" y1="36.068" x2="44.704" y2="33.528" width="0.4064" layer="1"/>
 </signal>
 <signal name="P2L.7">
 <contactref element="X6" pad="6"/>
-<contactref element="K15" pad="8"/>
 <via x="30.3403" y="27.3685" extent="1-16" drill="0.4" shape="octagon"/>
 <via x="30.3403" y="38.9128" extent="1-16" drill="0.4" shape="octagon"/>
 <wire x1="30.3403" y1="38.9128" x2="43.7769" y2="38.9128" width="0.4064" layer="16"/>
-<wire x1="43.7769" y1="38.9128" x2="44.704" y2="37.9857" width="0.4064" layer="16"/>
-<wire x1="44.704" y1="37.9857" x2="44.704" y2="36.068" width="0.4064" layer="16"/>
+<wire x1="43.7769" y1="38.9128" x2="44.958" y2="37.7317" width="0.4064" layer="16"/>
 <wire x1="30.3403" y1="27.3685" x2="18.9923" y2="27.3685" width="0.4064" layer="16"/>
 <wire x1="18.9923" y1="27.3685" x2="18.35" y2="27.285" width="0.4064" layer="16"/>
 <wire x1="30.3403" y1="38.9128" x2="30.3403" y2="27.3685" width="0.4064" layer="1"/>
+<contactref element="K17" pad="8"/>
+<wire x1="65.786" y1="36.068" x2="64.1223" y2="37.7317" width="0.4064" layer="16"/>
+<wire x1="64.1223" y1="37.7317" x2="44.958" y2="37.7317" width="0.4064" layer="16"/>
 </signal>
 <signal name="PORT_A0">
@@
 <wire x1="116.4463" y1="16.1544" x2="117.3607" y2="15.24" width="0.2032" layer="16"/>
 </signal>
-<signal name="P1">
+<signal name="P1.C">
 <contactref element="IC7" pad="8"/>
 <via x="117.9195" y="13.335" extent="1-16" drill="0.4" shape="octagon"/>
@@
 <wire x1="119.0371" y1="41.783" x2="117.8306" y2="41.783" width="0.2032" layer="1"/>
 </signal>
-<signal name="P2">
+<signal name="P2.C">
 <contactref element="IC8" pad="8"/>
 <contactref element="IC1" pad="43"/>

Commit message: Reed relay replacement
Parts:
- K1, K10, K11, K12, K13, K14, K15, K16, K17, K2, K3, K4, K5, K6, K7, K8, K9: value 3572.1220.051 -> HE721A0500
Changed lines of the file:
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@@
 <layer number="25" name="tNames" color="7" fill="1" visible="yes" active="yes"/>
 <layer number="26" name="bNames" color="5" fill="1" visible="no" active="yes"/>
-<layer number="27" name="tValues" color="14" fill="1" visible="no" active="yes"/>
+<layer number="27" name="tValues" color="14" fill="1" visible="yes" active="yes"/>
 <layer number="28" name="bValues" color="10" fill="1" visible="no" active="yes"/>
 <layer number="29" name="tStop" color="7" fill="1" visible="yes" active="yes"/>
@@
 <attribute name="VALUE" x="65" y="90.4925" size="1.27" layer="27" ratio="10" align="center"/>
 </element>
-<element name="K1" library="EEZ_switches" package="RR2A" value="3572.1220.051" x="31.242" y="52.324" smashed="yes" rot="R180">
+<element name="K1" library="EEZ_switches" package="RR2A" value="HE721A0500" x="31.242" y="52.324" smashed="yes" rot="R180">
 <attribute name="NAME" x="30.3784" y="55.3085" size="1.27" layer="25" ratio="10"/>
 <attribute name="VALUE" x="24.2824" y="51.5366" size="1.27" layer="27" ratio="10"/>
 </element>
-<element name="K3" library="EEZ_switches" package="RR2A" value="3572.1220.051" x="52.324" y="52.324" smashed="yes" rot="R180">
+<element name="K3" library="EEZ_switches" package="RR2A" value="HE721A0500" x="52.324" y="52.324" smashed="yes" rot="R180">
 <attribute name="NAME" x="51.3588" y="55.3974" size="1.27" layer="25" ratio="10"/>
 <attribute name="VALUE" x="45.5041" y="51.4985" size="1.27" layer="27" ratio="10"/>
 </element>
-<element name="K6" library="EEZ_switches" package="RR2A" value="3572.1220.051" x="73.406" y="52.324" smashed="yes" rot="R180">
+<element name="K6" library="EEZ_switches" package="RR2A" value="HE721A0500" x="73.406" y="52.324" smashed="yes" rot="R180">
 <attribute name="NAME" x="72.4154" y="55.3593" size="1.27" layer="25" ratio="10"/>
 <attribute name="VALUE" x="66.3067" y="51.6128" size="1.27" layer="27" ratio="10"/>
 </element>
-<element name="K8" library="EEZ_switches" package="RR2A" value="3572.1220.051" x="94.488" y="52.324" smashed="yes" rot="R180">
+<element name="K8" library="EEZ_switches" package="RR2A" value="HE721A0500" x="94.488" y="52.324" smashed="yes" rot="R180">
 <attribute name="NAME" x="93.5355" y="55.3466" size="1.27" layer="25" ratio="10"/>
 <attribute name="VALUE" x="87.5919" y="51.435" size="1.27" layer="27" ratio="10"/>
 </element>
-<element name="K12" library="EEZ_switches" package="RR2A" value="3572.1220.051" x="31.242" y="27.432" smashed="yes" rot="R180">
+<element name="K12" library="EEZ_switches" package="RR2A" value="HE721A0500" x="31.242" y="27.432" smashed="yes" rot="R180">
 <attribute name="NAME" x="30.226" y="30.3911" size="1.27" layer="25" ratio="10"/>
 <attribute name="VALUE" x="24.7142" y="26.5303" size="1.27" layer="27" ratio="10"/>
 </element>
-<element name="K14" library="EEZ_switches" package="RR2A" value="3572.1220.051" x="52.324" y="27.432" smashed="yes" rot="R180">
+<element name="K14" library="EEZ_switches" package="RR2A" value="HE721A0500" x="52.324" y="27.432" smashed="yes" rot="R180">
 <attribute name="NAME" x="51.4985" y="30.4927" size="1.27" layer="25" ratio="10"/>
 <attribute name="VALUE" x="45.6184" y="26.5684" size="1.27" layer="27" ratio="10"/>
 </element>
-<element name="K16" library="EEZ_switches" package="RR2A" value="3572.1220.051" x="73.406" y="27.432" smashed="yes" rot="R180">
+<element name="K16" library="EEZ_switches" package="RR2A" value="HE721A0500" x="73.406" y="27.432" smashed="yes" rot="R180">
 <attribute name="NAME" x="72.5932" y="30.4673" size="1.27" layer="25" ratio="10"/>
 <attribute name="VALUE" x="66.7258" y="26.6827" size="1.27" layer="27" ratio="10"/>
 </element>
-<element name="K2" library="EEZ_switches" package="RR2A" value="3572.1220.051" x="31.242" y="64.77" smashed="yes" rot="R180">
+<element name="K2" library="EEZ_switches" package="RR2A" value="HE721A0500" x="31.242" y="64.77" smashed="yes" rot="R180">
 <attribute name="NAME" x="29.6799" y="67.8815" size="1.27" layer="25" ratio="10"/>
 <attribute name="VALUE" x="24.384" y="64.1096" size="1.27" layer="27" ratio="10"/>
 </element>
-<element name="K4" library="EEZ_switches" package="RR2A" value="3572.1220.051" x="52.324" y="64.77" smashed="yes" rot="R180">
+<element name="K4" library="EEZ_switches" package="RR2A" value="HE721A0500" x="52.324" y="64.77" smashed="yes" rot="R180">
 <attribute name="NAME" x="50.5841" y="67.8815" size="1.27" layer="25" ratio="10"/>
 <attribute name="VALUE" x="45.4279" y="64.0207" size="1.27" layer="27" ratio="10"/>
 </element>
-<element name="K7" library="EEZ_switches" package="RR2A" value="3572.1220.051" x="73.406" y="64.77" smashed="yes" rot="R180">
+<element name="K7" library="EEZ_switches" package="RR2A" value="HE721A0500" x="73.406" y="64.77" smashed="yes" rot="R180">
 <attribute name="NAME" x="71.6026" y="67.8053" size="1.27" layer="25" ratio="10"/>
 <attribute name="VALUE" x="66.8274" y="64.0461" size="1.27" layer="27" ratio="10"/>
 </element>
-<element name="K10" library="EEZ_switches" package="RR2A" value="3572.1220.051" x="94.488" y="64.77" smashed="yes" rot="R180">
+<element name="K10" library="EEZ_switches" package="RR2A" value="HE721A0500" x="94.488" y="64.77" smashed="yes" rot="R180">
 <attribute name="NAME" x="92.8243" y="67.8053" size="1.27" layer="25" ratio="10"/>
 <attribute name="VALUE" x="87.8713" y="64.0207" size="1.27" layer="27" ratio="10"/>
 </element>
-<element name="K13" library="EEZ_switches" package="RR2A" value="3572.1220.051" x="31.242" y="39.878" smashed="yes" rot="R180">
+<element name="K13" library="EEZ_switches" package="RR2A" value="HE721A0500" x="31.242" y="39.878" smashed="yes" rot="R180">
 <attribute name="NAME" x="29.5656" y="42.8879" size="1.27" layer="25" ratio="10"/>
 <attribute name="VALUE" x="24.4348" y="39.1033" size="1.27" layer="27" ratio="10"/>
@@
 <attribute name="VALUE" x="114.3" y="39.243" size="1.27" layer="27" ratio="10" rot="R180" align="center"/>
 </element>
-<element name="K15" library="EEZ_switches" package="RR2A" value="3572.1220.051" x="52.324" y="39.878" smashed="yes" rot="R180">
+<element name="K15" library="EEZ_switches" package="RR2A" value="HE721A0500" x="52.324" y="39.878" smashed="yes" rot="R180">
 <attribute name="NAME" x="50.7111" y="42.8625" size="1.27" layer="25" ratio="10"/>
 <attribute name="VALUE" x="46.0756" y="39.0398" size="1.27" layer="27" ratio="10"/>
 </element>
-<element name="K17" library="EEZ_switches" package="RR2A" value="3572.1220.051" x="73.406" y="39.878" smashed="yes" rot="R180">
+<element name="K17" library="EEZ_switches" package="RR2A" value="HE721A0500" x="73.406" y="39.878" smashed="yes" rot="R180">
 <attribute name="NAME" x="71.8058" y="42.8371" size="1.27" layer="25" ratio="10"/>
 <attribute name="VALUE" x="66.8401" y="39.0779" size="1.27" layer="27" ratio="10"/>
 </element>
-<element name="K9" library="EEZ_switches" package="RR2A" value="3572.1220.051" x="31.242" y="77.216" smashed="yes" rot="R180">
+<element name="K9" library="EEZ_switches" package="RR2A" value="HE721A0500" x="31.242" y="77.216" smashed="yes" rot="R180">
 <attribute name="NAME" x="30.353" y="80.2894" size="1.27" layer="25" ratio="10"/>
 <attribute name="VALUE" x="38.0492" y="77.6605" size="1.27" layer="27" ratio="10" rot="R180"/>
 </element>
-<element name="K11" library="EEZ_switches" package="RR2A" value="3572.1220.051" x="73.406" y="77.216" smashed="yes" rot="R180">
+<element name="K11" library="EEZ_switches" package="RR2A" value="HE721A0500" x="73.406" y="77.216" smashed="yes" rot="R180">
 <attribute name="NAME" x="71.7931" y="80.3021" size="1.27" layer="25" ratio="10"/>
 <attribute name="VALUE" x="79.8703" y="77.4573" size="1.27" layer="27" ratio="10" rot="R180"/>
 </element>
-<element name="K5" library="EEZ_switches" package="RR2A" value="3572.1220.051" x="52.324" y="77.216" smashed="yes" rot="R180">
+<element name="K5" library="EEZ_switches" package="RR2A" value="HE721A0500" x="52.324" y="77.216" smashed="yes" rot="R180">
 <attribute name="NAME" x="53.1876" y="74.168" size="1.27" layer="25" ratio="10" rot="R180"/>
 <attribute name="VALUE" x="58.7629" y="77.6224" size="1.27" layer="27" ratio="10" rot="R180"/>
