File: EDA files/EEZ DIB MUX14D r1B3.brd (EAGLE design)
At the start: 131 x 95 mm, 65 parts, among them IC1 STM32F030C6T6, IC2 74HC1G126GW,125, IC3 M24C32-WMN6P, IC4 LP2985-33DBVR, IC5 MCP6001T-I/OT, IC6 LM335AZ, IC7 ULN2803ADWR, IC8 ULN2803ADWR, K1 HE721A0500, K10 HE721A0500, K11 HE721A0500, K12 HE721A0500, K13 HE721A0500, K14 HE721A0500, K15 HE721A0500, K16 HE721A0500, K17 HE721A0500, K2 HE721A0500, K3 HE721A0500, K4 HE721A0500, K5 HE721A0500, K6 HE721A0500, K7 HE721A0500, K8 HE721A0500, K9 HE721A0500, Q1 2N7002, X1 N.C., X2 77317-104-28LF, X3 DS1014-10RF1B, X4 DS1014-10RF1B, X5 691327310016, X6 691327310016

Commit message: Reed relay model correction
Parts:
- K1, K10, K11, K12, K13, K14, K15, K16, K17, K2, K3, K4, K6, K7, K8, K9: value HE721A0500 -> HE722A0500
Changed lines of the file:
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@@
 <attribute name="VALUE" x="65" y="90.4925" size="1.27" layer="27" ratio="10" align="center"/>
 </element>
-<element name="K1" library="EEZ_switches" package="RR2A" value="HE721A0500" x="31.242" y="52.324" smashed="yes" rot="R180">
+<element name="K1" library="EEZ_switches" package="RR2A" value="HE722A0500" x="31.242" y="52.324" smashed="yes" rot="R180">
 <attribute name="NAME" x="30.3784" y="55.3085" size="1.27" layer="25" ratio="10"/>
 <attribute name="VALUE" x="24.2824" y="51.5366" size="1.27" layer="27" ratio="10"/>
 </element>
-<element name="K3" library="EEZ_switches" package="RR2A" value="HE721A0500" x="52.324" y="52.324" smashed="yes" rot="R180">
+<element name="K3" library="EEZ_switches" package="RR2A" value="HE722A0500" x="52.324" y="52.324" smashed="yes" rot="R180">
 <attribute name="NAME" x="51.3588" y="55.3974" size="1.27" layer="25" ratio="10"/>
 <attribute name="VALUE" x="45.5041" y="51.4985" size="1.27" layer="27" ratio="10"/>
 </element>
-<element name="K6" library="EEZ_switches" package="RR2A" value="HE721A0500" x="73.406" y="52.324" smashed="yes" rot="R180">
+<element name="K6" library="EEZ_switches" package="RR2A" value="HE722A0500" x="73.406" y="52.324" smashed="yes" rot="R180">
 <attribute name="NAME" x="72.4154" y="55.3593" size="1.27" layer="25" ratio="10"/>
 <attribute name="VALUE" x="66.3067" y="51.6128" size="1.27" layer="27" ratio="10"/>
 </element>
-<element name="K8" library="EEZ_switches" package="RR2A" value="HE721A0500" x="94.488" y="52.324" smashed="yes" rot="R180">
+<element name="K8" library="EEZ_switches" package="RR2A" value="HE722A0500" x="94.488" y="52.324" smashed="yes" rot="R180">
 <attribute name="NAME" x="93.5355" y="55.3466" size="1.27" layer="25" ratio="10"/>
 <attribute name="VALUE" x="87.5919" y="51.435" size="1.27" layer="27" ratio="10"/>
 </element>
-<element name="K12" library="EEZ_switches" package="RR2A" value="HE721A0500" x="31.242" y="27.432" smashed="yes" rot="R180">
+<element name="K12" library="EEZ_switches" package="RR2A" value="HE722A0500" x="31.242" y="27.432" smashed="yes" rot="R180">
 <attribute name="NAME" x="30.226" y="30.3911" size="1.27" layer="25" ratio="10"/>
 <attribute name="VALUE" x="24.7142" y="26.5303" size="1.27" layer="27" ratio="10"/>
 </element>
-<element name="K14" library="EEZ_switches" package="RR2A" value="HE721A0500" x="52.324" y="27.432" smashed="yes" rot="R180">
+<element name="K14" library="EEZ_switches" package="RR2A" value="HE722A0500" x="52.324" y="27.432" smashed="yes" rot="R180">
 <attribute name="NAME" x="51.4985" y="30.4927" size="1.27" layer="25" ratio="10"/>
 <attribute name="VALUE" x="45.6184" y="26.5684" size="1.27" layer="27" ratio="10"/>
 </element>
-<element name="K16" library="EEZ_switches" package="RR2A" value="HE721A0500" x="73.406" y="27.432" smashed="yes" rot="R180">
+<element name="K16" library="EEZ_switches" package="RR2A" value="HE722A0500" x="73.406" y="27.432" smashed="yes" rot="R180">
 <attribute name="NAME" x="72.5932" y="30.4673" size="1.27" layer="25" ratio="10"/>
 <attribute name="VALUE" x="66.7258" y="26.6827" size="1.27" layer="27" ratio="10"/>
 </element>
-<element name="K2" library="EEZ_switches" package="RR2A" value="HE721A0500" x="31.242" y="64.77" smashed="yes" rot="R180">
+<element name="K2" library="EEZ_switches" package="RR2A" value="HE722A0500" x="31.242" y="64.77" smashed="yes" rot="R180">
 <attribute name="NAME" x="29.6799" y="67.8815" size="1.27" layer="25" ratio="10"/>
 <attribute name="VALUE" x="24.384" y="64.1096" size="1.27" layer="27" ratio="10"/>
 </element>
-<element name="K4" library="EEZ_switches" package="RR2A" value="HE721A0500" x="52.324" y="64.77" smashed="yes" rot="R180">
+<element name="K4" library="EEZ_switches" package="RR2A" value="HE722A0500" x="52.324" y="64.77" smashed="yes" rot="R180">
 <attribute name="NAME" x="50.5841" y="67.8815" size="1.27" layer="25" ratio="10"/>
 <attribute name="VALUE" x="45.4279" y="64.0207" size="1.27" layer="27" ratio="10"/>
 </element>
-<element name="K7" library="EEZ_switches" package="RR2A" value="HE721A0500" x="73.406" y="64.77" smashed="yes" rot="R180">
+<element name="K7" library="EEZ_switches" package="RR2A" value="HE722A0500" x="73.406" y="64.77" smashed="yes" rot="R180">
 <attribute name="NAME" x="71.6026" y="67.8053" size="1.27" layer="25" ratio="10"/>
 <attribute name="VALUE" x="66.8274" y="64.0461" size="1.27" layer="27" ratio="10"/>
 </element>
-<element name="K10" library="EEZ_switches" package="RR2A" value="HE721A0500" x="94.488" y="64.77" smashed="yes" rot="R180">
+<element name="K10" library="EEZ_switches" package="RR2A" value="HE722A0500" x="94.488" y="64.77" smashed="yes" rot="R180">
 <attribute name="NAME" x="92.8243" y="67.8053" size="1.27" layer="25" ratio="10"/>
 <attribute name="VALUE" x="87.8713" y="64.0207" size="1.27" layer="27" ratio="10"/>
 </element>
-<element name="K13" library="EEZ_switches" package="RR2A" value="HE721A0500" x="31.242" y="39.878" smashed="yes" rot="R180">
+<element name="K13" library="EEZ_switches" package="RR2A" value="HE722A0500" x="31.242" y="39.878" smashed="yes" rot="R180">
 <attribute name="NAME" x="29.5656" y="42.8879" size="1.27" layer="25" ratio="10"/>
 <attribute name="VALUE" x="24.4348" y="39.1033" size="1.27" layer="27" ratio="10"/>
@@
 <attribute name="VALUE" x="114.3" y="39.243" size="1.27" layer="27" ratio="10" rot="R180" align="center"/>
 </element>
-<element name="K15" library="EEZ_switches" package="RR2A" value="HE721A0500" x="52.324" y="39.878" smashed="yes" rot="R180">
+<element name="K15" library="EEZ_switches" package="RR2A" value="HE722A0500" x="52.324" y="39.878" smashed="yes" rot="R180">
 <attribute name="NAME" x="50.7111" y="42.8625" size="1.27" layer="25" ratio="10"/>
 <attribute name="VALUE" x="46.0756" y="39.0398" size="1.27" layer="27" ratio="10"/>
 </element>
-<element name="K17" library="EEZ_switches" package="RR2A" value="HE721A0500" x="73.406" y="39.878" smashed="yes" rot="R180">
+<element name="K17" library="EEZ_switches" package="RR2A" value="HE722A0500" x="73.406" y="39.878" smashed="yes" rot="R180">
 <attribute name="NAME" x="71.8058" y="42.8371" size="1.27" layer="25" ratio="10"/>
 <attribute name="VALUE" x="66.8401" y="39.0779" size="1.27" layer="27" ratio="10"/>
 </element>
-<element name="K9" library="EEZ_switches" package="RR2A" value="HE721A0500" x="31.242" y="77.216" smashed="yes" rot="R180">
+<element name="K9" library="EEZ_switches" package="RR2A" value="HE722A0500" x="31.242" y="77.216" smashed="yes" rot="R180">
 <attribute name="NAME" x="30.353" y="80.2894" size="1.27" layer="25" ratio="10"/>
 <attribute name="VALUE" x="38.0492" y="77.6605" size="1.27" layer="27" ratio="10" rot="R180"/>
 </element>
-<element name="K11" library="EEZ_switches" package="RR2A" value="HE721A0500" x="73.406" y="77.216" smashed="yes" rot="R180">
+<element name="K11" library="EEZ_switches" package="RR2A" value="HE722A0500" x="73.406" y="77.216" smashed="yes" rot="R180">
 <attribute name="NAME" x="71.7931" y="80.3021" size="1.27" layer="25" ratio="10"/>
 <attribute name="VALUE" x="79.8703" y="77.4573" size="1.27" layer="27" ratio="10" rot="R180"/>
